Commit message: Added python dd_man

File: ur5_robotiq3f_gazebo_ws/src/ur5/ur5_description/urdf/ur5_robotiq3f_gripper.urdf.xacro (robot description, xacro)
@@ -6,5 +6,5 @@
   <!-- <xacro:robotiq-3f-gripper_articulated prefix=""/> -->
   <joint name="gripper_tool0_joint" type="fixed">
-    <origin xyz="0 0 1" rpy="${-pi/2.0} ${-pi} ${-pi/2.0}" />
+    <origin xyz="0 0 0.005" rpy="${-pi/2.0} ${-pi} ${-pi/2.0}" />
     <parent link="tool0"/>
     <child link="palm"/>

File: ur5_robotiq3f_gazebo_ws/src/ur5_robotiq3f_moveit_config/config/gazebo_ur5.urdf (robot description, URDF)
Before this commit: robot ur5, 24 links, 23 joints
Joints:
- joint gripper_tool0_joint: origin xyz=0 0 0.07 rpy=-1.5707963267948966 -3.141592653589793 -1.5707963267948966 -> xyz=0 0 0.005 rpy=-1.5707963267948966 -3.141592653589793 -1.5707963267948966
