Commit message: Updated ur5_ws.

File: ur5_ws/src/dd_man/cabinet_models/my_cabinet/my_cabinet_test.urdf (robot description, URDF)
Before this commit: robot my_cabinet, 3 links, 2 joints
Links:
- link base_cabinet_link: geometry collision box size=0.018 0.346 0.546; collision box size=0.3 0.018 0.546
- link door_link: geometry collision box size=0.018 0.3 0.5; visual box size=0.018 0.3 0.5
Joints:
- joint joint_0: origin xyz=0.141 -0.117 0 -> xyz=0.141 -0.13999999999999999 0

Commit message: Green Summit ready.

File: ur5_ws/src/dd_man/cabinet_models/my_cabinet/my_cabinet_test.urdf (robot description, URDF)
Before this commit: robot my_cabinet, 3 links, 2 joints
Joints:
- removed joint virtual_joint
- added joint virtual_joint_cabinet: type fixed, parent world, child base_cabinet_link, origin xyz=0.0 0.0 0.0 rpy=0.0 0.0 0.0

File: ur5_ws/src/ur5_robotiq3f_moveit_config/config/gazebo_ur5.urdf (robot description, URDF)
Before this commit: robot ur5, 24 links, 23 joints
Links:
- added link camera_link
Joints:
- added joint camera_joint: type fixed, parent tool0, child camera_link, origin xyz=-0.1 0.0 0.0 rpy=0.0 0.0 -1.570796
- joint gripper_tool0_joint: origin xyz=0 0 0.005 rpy=-1.5707963267948966 -3.141592653589793 -1.5707963267948966 -> xyz=0 0 0.0535 rpy=-1.5707963267948966 -3.141592653589793 -1.5707963267948966
