Commit message: new moveit config

File: ferit_ur5_ws/src/ur5_configs/ur5_robotiq3f_moveit_config/config/gazebo_ur5.urdf (robot description, URDF)
Before this commit: robot ur5, 28 links, 27 joints
Links:
- removed link ft300_mounting_plate
- removed link ft300_sensor
Joints:
- removed joint ft300_fix
- removed joint ft300_mounting_plate
- joint gripper_joint: origin xyz=0 0 0 rpy=0 0 0 -> xyz=0 0 0.0535 rpy=-1.5707963267948966 -3.141592653589793 -1.5707963267948966; parent palm -> tool0
- joint gripper_tool0_joint: origin xyz=0 0 0.06 rpy=-1.5707963267948966 -3.141592653589793 -0.78539816339 -> xyz=0 0 0.0535 rpy=-1.5707963267948966 -3.141592653589793 -0.78539816339; parent ft300_sensor -> tool0
