Commit message: Latest updates. Latest tsr_data

File: ferit_ur5_ws/cabinet_handle_test.urdf (robot description, URDF)
Before this commit: robot my_cabinet, 4 links, 3 joints
Links:
- link base_cabinet_link: geometry collision box size=0.018 0.35423786141048347 0.4948382163542128; collision box size=0.4 0.018 0.4948382163542128
- link door_link: geometry collision box size=0.018 0.3082378614104835 0.4628382163542128; visual box size=0.018 0.3082378614104835 0.4628382163542128
Joints:
- joint door_joint: origin xyz=0.191 -0.12622267185648606 0.0 rpy=0.000000 -0.000000 3.141593 -> xyz=0.191 -0.14411893070524173 0.0 rpy=0.000000 -0.000000 3.141593
- joint handle_joint: origin xyz=-0.028999999999999998 -0.22244534371297214 0.0 rpy=0.000000 -0.000000 3.141593 -> xyz=-0.028999999999999998 -0.2582378614104835 0.0 rpy=0.000000 -0.000000 3.141593

Commit message: Fixed problems with script for running TSR experiments. Added checking forward kin in test_pkg. Added trajectories for 1000 experiments

File: ferit_ur5_ws/cabinet_handle_test.urdf (robot description, URDF)
Before this commit: robot my_cabinet, 4 links, 3 joints
Links:
- link base_cabinet_link: geometry collision box size=0.018 0.3461707579772326 0.4028860209979681; collision box size=0.4 0.018 0.4028860209979681
- link door_link: geometry collision box size=0.018 0.30017075797723264 0.3708860209979681; visual box size=0.018 0.30017075797723264 0.3708860209979681
Joints:
- joint door_joint: origin xyz=0.191 -0.14411893070524173 0.0 rpy=0.000000 -0.000000 3.141593 -> xyz=0.191 -0.1400853789886163 0.0 rpy=0.000000 -0.000000 3.141593
- joint handle_joint: origin xyz=-0.028999999999999998 -0.2582378614104835 0.0 rpy=0.000000 -0.000000 3.141593 -> xyz=-0.028999999999999998 -0.25017075797723265 0.0 rpy=0.000000 -0.000000 3.141593
