Commit message: Working on gazebo_push_open.

File: ferit_ur5_ws/cabinet.urdf (robot description, URDF)
Before this commit: robot my_cabinet, 3 links, 2 joints
Links:
- link base_cabinet_link: geometry collision box size=0.018 0.346 0.446; collision box size=0.35 0.018 0.446
Joints:
- removed joint joint_0
- added joint door_joint: type revolute, parent base_cabinet_link, child door_link, origin xyz=0.16599999999999998 0.13999999999999999 0 rpy=0 0 3.141592653589793, axis 0 0 1, limit lower=0 upper=1.5707963267948966 effort=50 velocity=10

Commit message: Updated README.md; Gazebo with one feasible pose ready.

File: ferit_ur5_ws/cabinet.urdf (robot description, URDF)
Before this commit: robot my_cabinet, 3 links, 2 joints
Links:
- link base_cabinet_link: geometry collision box size=0.018 0.346 0.546; collision box size=0.4 0.018 0.546
- link door_link: geometry collision box size=0.018 0.3 0.5; visual box size=0.018 0.3 0.5
Joints:
- joint door_joint: origin xyz=0.16599999999999998 0.13999999999999999 0 rpy=0 0 3.141592653589793 -> xyz=0.191 0.13999999999999999 0 rpy=0 0 3.141592653589793

File: ferit_ur5_ws/src/ur5_configs/ur5_robotiq3f_moveit_config/config/gazebo_ur5.urdf (robot description, URDF)
Before this commit: robot ur5, 25 links, 24 joints
Joints:
- joint finger_1_joint_1: origin xyz=0.020 0 0 rpy=0 0 0 -> xyz=0.020 0 0 rpy=0 -0.2 0
- joint finger_2_joint_1: origin xyz=0.020 0 0 rpy=0 0 0 -> xyz=0.020 0 0 rpy=0 0.2 0

Commit message: Tested real robot path planning

File: ferit_ur5_ws/cabinet.urdf (robot description, URDF)
Before this commit: robot my_cabinet, 3 links, 2 joints
Links:
- link base_cabinet_link: geometry collision box size=0.018 0.442 0.542; collision box size=0.3 0.018 0.542
- link door_link: geometry collision box size=0.018 0.396 0.496; visual box size=0.018 0.396 0.496
Joints:
- joint door_joint: limit lower=0 upper=1.5707963267948966 effort=50 velocity=10 -> lower=0 upper=-1.5707963267948966 effort=50 velocity=10; origin xyz=0.191 0.13999999999999999 0 rpy=0 0 0 -> xyz=0.141 -0.188 0 rpy=0 0 0

Commit message: Multi-contact final fixes. Running experiments...

File: ferit_ur5_ws/cabinet.urdf (robot description, URDF)
Before this commit: robot my_cabinet, 3 links, 2 joints
Links:
- added link handle_link, mass 0.050000; collision cylinder length=0.01 radius=0.003; collision cylinder length=0.02 radius=0.003
- link base_cabinet_link: geometry collision box size=0.018 0.3722537942019753 0.5851739159719982; collision box size=0.3 0.018 0.5851739159719982
- link door_link: geometry collision box size=0.018 0.3212537942019753 0.5391739159719982; visual box size=0.018 0.3212537942019753 0.5391739159719982
Joints:
- added joint handle_joint: type fixed, parent door_link, child handle_link, origin xyz=-0.028999999999999998 -0.2712537942019753 0.0 rpy=0.000000 -0.000000 3.141593
- joint door_joint: limit lower=0 upper=-1.5707963267948966 effort=50 velocity=10 -> lower=-1.658062789394613 upper=0 effort=50 velocity=10; origin xyz=0.191 -0.11508781744768028 0 rpy=0 0 0 -> xyz=0.141 -0.16062689710098765 0.0 rpy=0.000000 -0.000000 3.141593

File: ferit_ur5_ws/cabinet_handle_test.urdf (robot description, URDF)
Before this commit: robot my_cabinet, 4 links, 3 joints
Links:
- link base_cabinet_link: geometry collision box size=0.018 0.2932737136452283 0.4728399161172598; collision box size=0.3 0.018 0.4728399161172598
- link door_link: geometry collision box size=0.018 0.24227371364522832 0.42683991611725974; visual box size=0.018 0.24227371364522832 0.42683991611725974
Joints:
- joint door_joint: limit lower=0 upper=-1.5707963267948966 effort=50 velocity=10 -> lower=-1.658062789394613 upper=0 effort=50 velocity=10; origin xyz=0.191 -0.16221061243140697 0.0 rpy=0.000000 -0.000000 3.141593 -> xyz=0.141 -0.12113685682261416 0.0 rpy=0.000000 -0.000000 3.141593
- joint handle_joint: origin xyz=-0.028999999999999998 -0.29442122486281397 0.0 rpy=0.000000 -0.000000 3.141593 -> xyz=-0.028999999999999998 -0.19227371364522833 0.0 rpy=0.000000 -0.000000 3.141593

File: ferit_ur5_ws/src/ur5_configs/ur5_robotiq_ft_3f_moveit_config/config/gazebo_ur5_robotiq_ft_3f.urdf (robot description, URDF)
Before this commit: robot ur5_robotiq_ft_3f, 29 links, 28 joints
Links:
- link palm: geometry collision mesh filename=package://robotiq_3f_gripper_visualization/meshes/robotiq-3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; collision mesh filename=package://robotiq_3f_gripper_visualization/meshes/robotiq-3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
Joints:
- removed joint ft300_mounting_plate
- added joint ft300_mounting_plate_joint: type fixed, parent ft300_mounting_plate, child ft300_sensor, origin xyz=0 0 0.0415 rpy=0 3.141592653589793 0

Commit message: Added RVL data

File: ferit_ur5_ws/cabinet.urdf (robot description, URDF)
Before this commit: robot my_cabinet, 4 links, 3 joints
Links:
- removed link handle_link
- link base_cabinet_link: geometry collision box size=0.018 0.448 0.529; collision box size=0.4 0.018 0.529
- link door_link: geometry collision box size=0.018 0.397 0.483; visual box size=0.018 0.397 0.483
Joints:
- removed joint handle_joint
- joint door_joint: origin xyz=0.141 -0.16062689710098765 0.0 rpy=0.000000 -0.000000 3.141593 -> xyz=0.191 -0.1985 0.0 rpy=0.000000 -0.000000 3.141593
