Commit message: Added door replanning based on sensor fusion

File: ferit_ur5_ws/cabinet_new.urdf (robot description, URDF)
Before this commit: robot my_cabinet, 4 links, 3 joints
Links:
- removed link handle_link
Joints:
- removed joint handle_joint

File: ferit_ur5_ws/src/ur5_configs/fmauch_universal_robot/ur_description/urdf/ur5_robotiq_ft_3f.urdf.xacro (robot description, xacro)
@@ -35,7 +35,41 @@
   </joint>
   <joint name="gripper_coupler_robotiq_3f_joint" type="fixed">
-    <origin xyz="0 0 ${0.0535 + 0.0065}" rpy="${pi/2.0} ${0} ${-pi/4.0}" />
+    <!-- <origin xyz="0 0 ${0.0535 + 0.0065}" rpy="${pi/2.0} ${0} ${-pi/4.0}" /> -->
+    <origin xyz="0 0 ${0.0535 + 0.013 + 0.004}" rpy="${pi/2.0} ${0} ${-pi/4.0}" />
     <parent link="gripper_coupler"/>
     <child link="palm"/>
+  </joint>
+  <link name="camera_link">
+      <visual>
+          <origin rpy="0 0 0" xyz="0 0 0" />
+          <geometry>
+              <mesh filename="package://intel_realsense_l515/meshes/visual/l515.stl" />
+          </geometry>
+          <material name="yellow">
+              <color rgba="1 1 0 1" />
+          </material>
+      </visual>
+      <collision>
+          <origin rpy="0 0 0" xyz="0 0 0" />
+          <geometry>
+              <mesh filename="package://intel_realsense_l515/meshes/collision/l515.stl" />
+          </geometry>
+      </collision>
+      <inertial>
+      <origin xyz="0 0 0" rpy="0 0 0"/>
+      <mass value="0.3"/>
+      <inertia
+          ixx="0.0001027"
+          ixy="0.0"
+          ixz="0.0"
+          iyy="0.0001027"
+          iyz="0.0"
+          izz="0.0001442"/>
+      </inertial>
+  </link>
+  <joint name="camera_joint" type="fixed">
+      <origin rpy="0.0033192 -0.0293569 2.3598604" xyz="-0.07941524 -0.08149755 0.0608904" />
+      <parent link="tool0" />
+      <child link="camera_link" />
   </joint>
   <link name="world" />

File: ferit_ur5_ws/src/ur5_configs/ur5_robotiq_ft_3f_moveit_config/config/gazebo_ur5_robotiq_ft_3f.urdf (robot description, URDF)
Before this commit: robot ur5_robotiq_ft_3f, 29 links, 28 joints
Links:
- added link camera_link, mass 0.3; collision mesh filename=package://intel_realsense_l515/meshes/collision/l515.stl; visual mesh filename=package://intel_realsense_l515/meshes/visual/l515.stl
Joints:
- added joint camera_joint__: type fixed, parent tool0, child camera_link, origin xyz=-0.07941524 -0.08149755 0.0608904 rpy=0.0033192 -0.0293569 -0.7817323
