Commit message: Updated stuff

File: Helper3D-master/robotiq-3f-gripper_articulated_collision.urdf (robot description, URDF)
Before this commit: robot robotiq-3f-gripper_articulated, 13 links, 12 joints
Links:
- link palm: geometry collision mesh filename=/home/RVLuser/ferit_ur5_ws/src/ur5_configs/robotiq-noetic-d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; visual mesh filename=/home/RVLuser/ferit_ur5_ws/src/ur5_configs/robotiq-noetic-d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
